File: PCB/SEM_Display/SEM_Display.kicad_pcb (KiCad board)
At the start: 2 copper layers, 83.8 x 68.6 mm, 23 parts, among them IC1 LD1117V33, J1 Conn_01x04_Pin, J2 Conn_01x04_Pin, J3 Conn_01x03_Pin, J4 Conn_01x04_Pin, J5 Conn_01x02_Pin, SW1 SW_Push, SW2 SW_Push, SW3 SW_Push, SW4 SW_Push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

Commit message: Converted Global Dependencies into local ones
Parts:
- U1: footprint Espressif:ESP32-WROVER-E -> Espresif:ESP32-WROVER-E
Changed lines of the file:
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@@
   (net 31 "unconnected-(U1-GND_THERMAL-Pad39)")
   (net 32 "unconnected-(U2-BLK-Pad7)")
-  (footprint "Espressif:ESP32-WROVER-E" (layer "F.Cu")
+  (footprint "Espresif:ESP32-WROVER-E" (layer "F.Cu")
     (at 100.47 92.075)
     (descr "ESP32-WROVER-E: https://www.espressif.com/sites/default/files/documentation/esp32-wroom-32e_esp32-wroom-32ue_datasheet_en.pdf")
