File: PCB/SEM_Display/SEM_Display.kicad_sch (KiCad schematic)
At the start: 23 parts, among them IC1 LD1117V33, J1 Conn_01x04_Pin, J2 Conn_01x04_Pin, J3 Conn_01x03_Pin, J4 Conn_01x04_Pin, J5 Conn_01x02_Pin, SW1 SW_Push, SW2 SW_Push, SW3 SW_Push, SW4 SW_Push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

Commit message: Converted Global Dependencies into local ones
Parts:
- IC1: symbol SamacSys_Parts:LD1117V33 -> SamacSys_parts:LD1117V33
- U1: footprint Espressif:ESP32-WROVER-E -> Espresif:ESP32-WROVER-E
Other:
- note added: "Prog Inputs"
Changed lines of the file:
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@@
     (effects (font (size 1.27 1.27)) (justify left bottom))
   )
-  (text "Control Inputs\n" (at 76.2 16.51 0)
+  (text "Prog Inputs\n" (at 76.2 16.51 0)
     (effects (font (size 1.27 1.27)) (justify left bottom))
   )
@@
       (effects (font (size 1.27 1.27)) (justify left))
     )
-    (property "Footprint" "Espressif:ESP32-WROVER-E" (at 95.25 115.57 0)
+    (property "Footprint" "Espresif:ESP32-WROVER-E" (at 95.25 115.57 0)
       (effects (font (size 1.27 1.27)) hide)
     )
@@
     )
   )
-  (symbol (lib_id "SamacSys_Parts:LD1117V33") (at 226.06 140.97 0) (unit 1)
+  (symbol (lib_id "SamacSys_parts:LD1117V33") (at 226.06 140.97 0) (unit 1)
     (in_bom yes) (on_board yes) (dnp no) (fields_autoplaced)
     (property "Reference" "IC1" (at 250.19 142.875 0)
